Commit message: Turned on torque limit command guard, path to joint_limits made configurable (xacro argument).

File: lbr_description/urdf/iiwa7/iiwa7_description.xacro (robot description, xacro)
@@ -8,6 +8,6 @@
         <xacro:include filename="$(find lbr_description)/ros2_control/lbr_system_interface.xacro" />
         <!-- joint limits via yaml -->
-        <xacro:property name="joint_limits_path"
-            value="$(find lbr_description)/urdf/iiwa7/joint_limits.yaml" />
+        <xacro:arg name="joint_limits_path" default="$(find lbr_description)/urdf/iiwa7/joint_limits.yaml" />
+        <xacro:property name="joint_limits_path" value="$(arg joint_limits_path)" />
         <xacro:property name="joint_limits" value="${xacro.load_yaml(joint_limits_path)}" />
         <!-- constants -->
